File: JIG_EXTENSION.kicad_pcb (KiCad board)
At the start: 2 copper layers, 180 x 180 mm, 116 parts, among them J10 USB_B, J11 VIN, J12 Conn_01x02_Pin, J13 Conn_01x02_Pin, J14 Conn_01x02_Pin, J15 Conn_01x02_Pin, J16 Conn_01x02_Pin, J17 VIN, J18 Conn_01x04_Pin, J19 Conn_01x04_Pin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

Commit message: saveddddd
Parts:
- added C15: 10uF, Capacitor_SMD:C_1206_3216Metric, F.Cu at (197.0, 175.8)
- added C16: 10uF, Capacitor_SMD:C_1206_3216Metric, F.Cu at (197.4, 190.8)
- added J1: Conn_01x02_Pin, Connector_PinHeader_2.54mm:PinHeader_1x02_P2.54mm_Vertical, F.Cu at (189.8, 176.7)
- added J2: Conn_01x02_Pin, Connector_PinHeader_2.54mm:PinHeader_1x02_P2.54mm_Vertical, F.Cu at (190.0, 192.0)
- added Q4: WST4041, Package_TO_SOT_SMD:SOT-23, F.Cu at (258.5, 198.0)
- added Q7: WST2303, Package_TO_SOT_SMD:SOT-23, F.Cu at (265.0, 198.0)
- added R51: 0, Resistor_SMD:R_0603_1608Metric, F.Cu at (250.2, 200.6)
- added R52: 0, Resistor_SMD:R_0603_1608Metric, F.Cu at (259.6, 202.7)
- added R62: 20K, Resistor_SMD:R_0603_1608Metric, F.Cu at (254.8, 197.9)
- added R63: 1K, Resistor_SMD:R_0603_1608Metric, F.Cu at (269.4, 196.0)
- added R64: 0, Resistor_SMD:R_0603_1608Metric, F.Cu at (269.4, 199.0)
- added R65: 3K3, Resistor_SMD:R_0603_1608Metric, F.Cu at (242.8, 200.6)
- added R66: 3K3, Resistor_SMD:R_0603_1608Metric, F.Cu at (246.4, 200.6)
- added R67: 0, Resistor_SMD:R_0603_1608Metric, F.Cu at (197.2, 183.2)
- added R68: 0, Resistor_SMD:R_0603_1608Metric, F.Cu at (197.4, 197.6)
- added U5: LMV331, Package_TO_SOT_SMD:SOT-23-5, F.Cu at (197.2, 180.0)
- added U6: LMV331, Package_TO_SOT_SMD:SOT-23-5, F.Cu at (197.4, 194.4)
- moved R57 78.0 mm to (301.3, 192.4)
- moved R33 59.6 mm to (213.3, 70.3)
- moved C13 59.6 mm to (221.5, 70.1)
- moved Q2 59.6 mm to (222.3, 62.6)
- moved R60 59.6 mm to (226.3, 60.7)
- moved U4 59.6 mm to (243.9, 63.5)
- moved C14 59.6 mm to (219.1, 71.7)
- moved C5 59.6 mm to (252.8, 59.6)
- moved C6 59.6 mm to (238.1, 58.9)
- moved D1 59.6 mm to (253.1, 72.2)
- moved D10 59.6 mm to (217.3, 57.4)
- moved D11 59.6 mm to (217.2, 60.1)
- moved D5 59.6 mm to (256.9, 60.0)
- moved D6 59.6 mm to (192.1, 68.7)
- moved D7 59.6 mm to (192.1, 59.7)
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Connections:
- J7 pad 28: unconnected-(J7-Pad28) -> /DB_28
- J7 pad SHELL: Net-(J7-PadSHELL) -> unconnected-(J7-PadSHELL)
- J7 pad SHELL1: Net-(J7-PadSHELL) -> unconnected-(J7-PadSHELL)
- R14 pad 1: /AI3 -> /EBL
- U1 pad 21: unconnected-(U1-D32-Pad21) -> Net-(U1-D32)
Routing:
- net Net-(U1-D32): track 0.00 -> 203.7 mm, vias 0 -> 1
- net +12V: track 322.2 -> 510.1 mm
- net /DB_28: track 0.00 -> 157.1 mm, vias 0 -> 3
- net 3V3_B: track 277.9 -> 408.6 mm, vias 3 -> 4
- net unconnected-(U1-D34-Pad19): track 116.3 -> 0.00 mm, vias 2 -> 0
- net 5V0: track 246.1 -> 340.4 mm, vias 3 -> 7
- net Net-(J7-PadSHELL): track 87.9 -> 0.00 mm
- net /AI7: track 0.00 -> 77.2 mm, vias 0 -> 3
- net /DB_16: track 87.1 -> 162.1 mm
- net unconnected-(J7-PadSHELL): track 0.00 -> 72.1 mm
- net 3V3: track 158.5 -> 90.0 mm
- net /D+/A: track 191.7 -> 126.6 mm
- net /D-/B: track 189.2 -> 125.8 mm
- net /UART_RS485_RX: track 176.8 -> 117.9 mm
- net /MOSI: track 71.2 -> 33.1 mm, vias 4 -> 2
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Other:
- board size 180 x 180 mm -> 180 x 155 mm
- board text added: "DB37 20 21 22 23 24 25 26 27 28"
- board text added: "DUT 12V IN"
- board text added: "Pin_Description SWDCLK VCU_SWDIO VCU_SWCLK GPIO_2 GPIO_3 GPIO_4 AIN_100V GND T_BAT"
- board text added: "ROAM JIG V1.1"
- board text added: "Test_PIN J7-11 J7-12 J7-13 J7-14 J7-15 J7-16 J7-17 J7-18 TP9"
- board text removed: "DB37 20 21 22 23 24 25 26 27"
- board text removed: "Pin_Description SWDCLK VCU_SWDIO VCU_SWCLK GPIO_2 GPIO_3 GPIO_4 AIN_100V GND"
- board text removed: "ROAM JIG V1.0"
- board text removed: "Test_PIN J7-11 J7-12 J7-13 J7-14 J7-15 J7-16 J7-17 J7-18"
- board text removed: "UART2 EXTERNAL"

Commit message: UPDATE BOM
Parts:
- added D12: SS34F, Diode_SMD:D_SMA, F.Cu at (264.0, 133.7)
- added D13: SS34F, Diode_SMD:D_SMA, F.Cu at (284.4, 119.3)
- added R69: 0, Resistor_SMD:R_0603_1608Metric, F.Cu at (272.8, 108.3)
- C1, C13, C4: value 100n -> 100nF
- Q7: value WST2303 -> BC846
- R45: value 2k -> 2K
- R62: value 20K -> 820
- U11: footprint footprint:SOIC127P600X175-8N -> YZ-Audio:SOIC127P600X175-8N
- U5, U6: value LMV331 -> LMV321
Connections:
- net Net-(J10-VBUS) renamed 5V0_VBUS_CONBINE
- J7 pad 34: unconnected-(J7-Pad34) -> /AI15
- J7 pad 35: unconnected-(J7-Pad35) -> /UART_ESP_NRF_FOR_BLACK
- J7 pad 36: unconnected-(J7-Pad36) -> /EXT_BTN
- J7 pad 37: unconnected-(J7-Pad37) -> /3V3_FOR_BLACK
- R1 pad 2: /UART_QT_RX -> /UART_ESP_NRF_FOR_BLACK
- R19 pad 2: /UART_QT_RX -> /UART_ESP_NRF_FOR_BLACK
- R21 pad 2: /UART_QT_RX -> /UART_ESP_NRF_FOR_BLACK
- U1 pad 5: unconnected-(U1-D4-Pad5) -> Net-(U1-D4)
Routing:
- net /AI15: track 0.00 -> 176.7 mm, vias 0 -> 2
- net /UART_ESP_NRF_FOR_BLACK: track 0.00 -> 165.3 mm, vias 0 -> 2
- net /EXT_BTN: track 0.00 -> 126.2 mm, vias 0 -> 2
- net /3V3_FOR_BLACK: track 0.00 -> 115.9 mm
- net /UART_QT_RX: track 73.7 -> 0.00 mm
- net 5V0_VBUS_CONBINE: track 39.8 -> 85.7 mm
- net 5V0: track 340.4 -> 373.9 mm
- net 3V3: track 90.0 -> 104.4 mm, vias 3 -> 4
- net Net-(U1-D4): track 0.00 -> 4.70 mm
Other:
- board text added: "BLACK JIG V1.0"
- board text added: "DB37 20 21 22 23 24 25 26 27 28 29 30 31 32 33 34 35 36 37"
- board text removed: "DB37 20 21 22 23 24 25 26 27 28"
- board text removed: "Pin_Description 4V7_BOOST 5V0 UART_TX 60VIN 3V3_ALWAYS_ON UART_RX EBL 4V0_MODEM 3V3_ANT 60V CAN_250_H CAN_250_L CAN_500_H CAN_500_L IM_OUT GPIO_5 GPIO_1 TAMPER_CONN SWDIO"
- board text removed: "Pin_Description SWDCLK VCU_SWDIO VCU_SWCLK GPIO_2 GPIO_3 GPIO_4 AIN_100V GND T_BAT"
- board text removed: "ROAM JIG V1.1"
- board text removed: "Test_PIN J7-11 J7-12 J7-13 J7-14 J7-15 J7-16 J7-17 J7-18 TP9"
- board text removed: "Test_PIN TP1 TP2 TP3 TP4 TP5 TP6 TP7 TP8 TP10 J7-1 J7-2 J7-3 J7-4 J7-5 J7-6 J7-7 J7-8 J7-9 J7-10"
