File: JIG_EXTENSION.kicad_sch (KiCad schematic)
At the start: 114 parts, among them J1 Conn_01x03_Pin, J10 USB_B, J11 VIN, J12 Conn_01x02_Pin, J13 Conn_01x02_Pin, J14 Conn_01x02_Pin, J15 Conn_01x02_Pin, J16 Conn_01x02_Pin, J17 VIN, J18 Conn_01x04_Pin, J19 Conn_01x04_Pin, J20 Conn_01x04_Pin, J21 VIN, J22 Conn_02x04_Odd_Even, J3 Conn_01x07_Pin, J4 Conn_01x12_Socket, J5 Conn_01x12_Socket, J6 VIN, J7 618037231321, J8 Conn_01x18_Pin, J9 Conn_01x19_Pin, Q1 WST3325, U1 ESP32-DEVKIT-V1, U10 MCP2562-E-MF, U11 MAX13487EESAT, U2 CH340E, U3 AMS1117-3.3, U4 NCP1117DT50RKG, U5 SN74LVC1G3157DBVR, U6 SN74LVC1G3157DBVR, U9 MCP2515-xST, Y1 16MHz

Commit message: 1,1
Parts:
- added JP1, JP2: SolderJumper_2_Open, Jumper:SolderJumper-2_P1.3mm_Open_RoundedPad1.0x1.5mm, symbol Jumper:SolderJumper_2_Open
- added Q2, Q3: MMBT3904, Package_TO_SOT_SMD:SOT-23, symbol Transistor_BJT:MMBT3904
- added R57: 0, Resistor_SMD:R_0603_1608Metric, symbol Device:R
- added R58, R59: 10k, Resistor_SMD:R_0603_1608Metric, symbol Device:R_Small
- added R60, R61: 1K, Resistor_SMD:R_0603_1608Metric, symbol Device:R_Small
- D10, D11: footprint LED_SMD:LED_0805_2012Metric -> LED_SMD:LED_0603_1608Metric
- J1: footprint Connector_JST:JST_XH_S3B-XH-A_1x03_P2.50mm_Horizontal -> Connector_PinSocket_2.54mm:PinSocket_1x03_P2.54mm_Horizontal
- R53, R54: value 1K -> 2K
Connections:
- net +12V: now also R57.1
- net 3V3: now also R58.2, R59.2, R60.2; no longer C13.1, C14.1, D10.2 (A), D11.2 (A), R32.2, R33.2, R34.2, R35.2, R40.2, R41.2, U11.8 (VCC)
- net 5V0: now also C13.1, C14.1, D10.2 (A), D11.2 (A), R32.2, R33.2, R34.2, R35.2, R40.2, R41.2, U11.8 (VCC), R61.2
- net DB_10: now also R57.2
- net UART_RS485_RX: now also JP2.1 (A), Q2.2 (E), R58.1; no longer R34.1, R54.2, U11.4 (DI)
- net UART_RS485_TX: now also JP1.1 (A), Q3.3 (C), R59.1; no longer R32.1, R53.2, U11.1 (RO)
- new net: Q3.1 (B), R61.1
- new net: Q2.1 (B), R60.1
- new net UART_RS485_RX_5V: JP2.2 (B), Q2.3 (C), R34.1, R53.2, U11.4 (DI)
- new net UART_RS485_TX_5V: JP1.2 (B), Q3.2 (E), R32.1, R54.2, U11.1 (RO)
Other:
- moved on the sheet: C10, C11, C12, C13, C14, C5, C6, C7, C8, C9, D1, D10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

Commit message: delete jlink selector
Parts:
- removed J20: Conn_01x04_Pin, Connector_PinHeader_2.54mm:PinHeader_1x04_P2.54mm_Horizontal, symbol Connector:Conn_01x04_Pin
- removed R52: 10K, Resistor_SMD:R_0603_1608Metric, symbol Device:R_Small
- removed U5, U6: SN74LVC1G3157DBVR, Package_TO_SOT_SMD:SOT-23-6, symbol SN74LVC1G3157DBVR:SN74LVC1G3157DBVR
Other:
- note removed: "B1 set low to enable"

Commit message: saveddddd
Parts:
- removed J1: Conn_01x03_Pin, Connector_PinSocket_2.54mm:PinSocket_1x03_P2.54mm_Horizontal, symbol Connector:Conn_01x03_Pin
- removed J22: Conn_02x04_Odd_Even, Connector_PinHeader_2.54mm:PinHeader_2x04_P2.54mm_Horizontal, symbol Connector_Generic:Conn_02x04_Odd_Even
- removed J3: Conn_01x07_Pin, Connector_PinSocket_2.54mm:PinSocket_1x07_P2.54mm_Vertical, symbol Connector:Conn_01x07_Pin
- added C15, C16: 10uF, Capacitor_SMD:C_1206_3216Metric, symbol Device:C
- added J1, J2: Conn_01x02_Pin, Connector_PinHeader_2.54mm:PinHeader_1x02_P2.54mm_Vertical, symbol Connector:Conn_01x02_Pin
- added Q4: WST4041, Package_TO_SOT_SMD:SOT-23, symbol Device:Q_PMOS_GSD
- added Q7: WST2303, Package_TO_SOT_SMD:SOT-23, symbol Transistor_FET:2N7002E
- added R52, R64, R67, R68: 0, Resistor_SMD:R_0603_1608Metric, symbol Device:R
- added R62: 20K, Resistor_SMD:R_0603_1608Metric, symbol Device:R
- added R63: 1K, Resistor_SMD:R_0603_1608Metric, symbol Device:R
- added R65, R66: 3K3, Resistor_SMD:R_0603_1608Metric, symbol Device:R
- added U5, U6: LMV331, Package_TO_SOT_SMD:SOT-23-5, symbol Comparator:LMV331
Connections:
- net SWD_SEL is gone; now on net DB_15: R51.2
- net +12V: now also Q4.2 (S), R62.2, R65.2
- net 5V0: now also C15.1, C16.1, U5.5 (V+), U6.5 (V+)
- net AI3: now also J1.2 (Pin_2), R67.1, U5.3 (-); no longer R14.1
- net AI6: now also J2.2 (Pin_2), R68.1, U6.3 (-)
- net AI7: now also R65.1, R66.2
- net DB_16: now also R52.2
- net DB_28: now also J7.28, J2.1 (Pin_1), U6.1 (+)
- net GND: now also C15.2, C16.2, R63.1, U5.2 (V-), U6.2 (V-)
- net at U1.19 (D34): no longer R51.1
- net at U1.21 (D32): now also R64.1
- new net: Q4.1 (G), Q7.3 (D), R62.1
- new net: R67.2, U5.4
- new net: Q7.2 (S), R63.2
- new net: R68.2, U6.4
- new net EBL: J1.1 (Pin_1), R14.1, U5.1 (+)
- new net GPIO_5: Q4.3 (D), R52.1
- new net GPIO_5_CON: Q7.1 (G), R64.2
- new net IM_OUT: R51.1, R66.1
- no-connect marks 11 -> 34
Other:
- moved on the sheet: C10, C11, C12, C13, C14, C7, C8, C9, D10, D11, D2, D6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

Commit message: UPDATE BOM
Parts:
- added D12, D13: SS34F, Diode_SMD:D_SMA, symbol Device:D
- added R69: 0, Resistor_SMD:R_0603_1608Metric, symbol Device:R
- C1, C13, C4: value 100n -> 100nF; JLC PN (none) -> C14663; MPN (none) -> CC0603KRX7R9BB104
- C10, C9: JLC PN (none) -> C14663; MPN 06036C104KAT4A -> CC0603KRX7R9BB104
- C11, C8: JLC PN (none) -> C1647; MPN 251R14S180JV4T -> 18pF ±5% 50V
- C12: JLC PN (none) -> C1523; MPN 0402N102F500CT -> 1nF ±10% 50V
- C14, C2, C3: JLC PN (none) -> C15849; MPN (none) -> CL10A105KB8NNNC
- C15, C16, C5: JLC PN (none) -> C13585; MPN (none) -> 10uF ±10% 50V
- C6, C7: JLC PN (none) -> C96446; MPN (none) -> 10uF ±20% 25V
- D1, D3, D4, D8, D9: JLC PN (none) -> C84256; MPN 0805RBD0070S01 -> 红灯 0805红灯 正贴
- D10, D11: JLC PN (none) -> C496822; MPN 0805RBD0070S01 -> (none)
- D2: JLC PN (none) -> C1973833
- D5: JLC PN (none) -> C550954; MPN BZX84B4V7LT1 -> BZX84-C4V7,235
- D6, D7: JLC PN (none) -> C2920017; MPN (none) -> P6SMB6.8CA
- F2: JLC PN (none) -> C140468; MPN C1F 2 -> 贴片式保险丝
- J1, J12, J13, J14, J15, J16, J2: JLC PN (none) -> C492401; MPN (none) -> 间距:2.54mm 1x2P 直插 方针 【排针】
- J10: JLC PN (none) -> C2962393; MPN (none) -> 【插件】Type-B 母座 弯插
- J11, J17, J21, J6: JLC PN (none) -> C8475; MPN (none) -> 5mm 1x2P 排数:1 每排P数:2 直针 可拼接【螺钉】
- J18, J19: JLC PN (none) -> C492467; MPN (none) -> 间距:2.5mm 1x4P 弯插 【插件】
- J4, J5: JLC PN (none) -> C225409; MPN (none) -> 系列:XH 间距:2.5mm 1x12P 镀锡【插件】
- J7: JLC PN (none) -> C5156644; MPN (none) -> D-SUB-DR-37FKSM
- J8: JLC PN (none) -> C725950; MPN (none) -> 间距:2.54mm 1x18P 直插 方针 高镀金 抗氧化【排针】
- J9: JLC PN (none) -> C725951; MPN (none) -> 间距:2.54mm 1x19P 直插 方针 高镀金 抗氧化【排针】
- JP1, JP2: JLC PN (none) -> DNP
- Q1: JLC PN (none) -> C148355; MPN NTR3A30PZT1G -> WST3325
- Q2, Q3: JLC PN (none) -> C20526; MPN (none) -> MMBT3904
- Q4: JLC PN (none) -> C148357; MPN (none) -> WST4041
- Q7: value WST2303 -> BC846; symbol Transistor_FET:2N7002E -> Transistor_BJT:BC846; JLC PN (none) -> C779722; MPN (none) -> BC846
- R1, R11, R12, R13, R14, R15, R16, R17, R18, R19, R2, R20, R3, R31, R4, R42, R43, R44, R47, R48, R49, R5, R50, R51, R52, R55, R56, R57, R6, R64, R67, R68, R7, R8, R9: JLC PN (none) -> C21189; MPN (none) -> 0603WAF0000T5E
- R10: JLC PN (none) -> C3202451; MPN (none) -> TR0603B5K00P0525Z
- R21, R22, R46, R60, R61, R63: JLC PN (none) -> C21190; MPN (none) -> 0603WAF1001T5E
- R23: JLC PN (none) -> C25803; MPN (none) -> 0603WAF1003T5E
- R24, R25: JLC PN (none) -> C25804; MPN RMCF0603FT10K0CT-ND -> 0603WAF1002T5E
- R26, R27: JLC PN (none) -> C17168; MPN RMCF0402ZT0R00 -> 0402WGF0000TCE
- R28, R29: JLC PN (none) -> C861820; MPN RC0603FR-072K8L -> RT0603BRE072K8L
- R30, R37, R40, R41: JLC PN (none) -> DNP; MPN (none) -> DNP
- R32, R33, R34, R58, R59: JLC PN (none) -> C25804; MPN (none) -> 0603WAF1002T5E
- R35, R36: JLC PN (none) -> C23162; MPN (none) -> 0603WAF4701T5E
- R38, R39: JLC PN (none) -> C17902; MPN (none) -> 1206W4F1002T5E
- R45: value 2k -> 2K; JLC PN (none) -> C22975; MPN (none) -> 0603WAF2001T5E
- R53, R54: JLC PN (none) -> C22975; MPN (none) -> 0603WAF2001T5E
- R62: value 20K -> 820; JLC PN (none) -> C23253; MPN (none) -> 0603WAF8200T5E
- R65, R66: JLC PN (none) -> C22978; MPN (none) -> 0603WAF3301T5E
- U10: JLC PN (none) -> C635113; MPN MCP2562-E-MF -> MCP2562-E/MF
- U11: JLC PN (none) -> C18347; MPN (none) -> MAX13487EESA+T
- U2: JLC PN (none) -> C99652; MPN (none) -> CH340E
- U3: JLC PN (none) -> C6186; MPN (none) -> AMS1117-3.3
- U4: JLC PN (none) -> C152470; MPN (none) -> NCP1117DT50RKG
- U5, U6: value LMV331 -> LMV321; JLC PN (none) -> C395459; MPN (none) -> LMV321
- U9: JLC PN (none) -> C185941; MPN MCP2515-I/ST -> MCP2515-xST
- Y1: JLC PN (none) -> C70562; MPN ABM8-16.000MHZ-D1X-T -> X322516MRB4SI
Connections:
- net UART_QT_RX is gone; now on net UART_ESP_NRF_FOR_BLACK: R1.2, R19.2, R21.2
- net 3V3: now also D12.2 (A)
- net 5V0: now also D13.2 (A)
- net AI15: now also J7.34
- net 5V0_VBUS_CONBINE: now reaches C1.1, C2.1, J10.1 (VBUS), U3.3 (VI)
- net 5V0_VBUS_CONBINE: now also D13.1 (K)
- net UART_ESP_NRF_FOR_BLACK: now reaches J7.35
- net EXT_BTN: now reaches J7.36
- net EXT_BTN: now also R69.1
- net 3V3_FOR_BLACK: now reaches J7.37
- net 3V3_FOR_BLACK: now also D12.1 (K)
- net at U1.5 (D4): now also R69.2
- no-connect marks 34 -> 29
Other:
- note added: "3V3_DETECT_FOR_BALCK"
- note added: "Bypass the 5V to VBUS."
- note added: "Pin_Description 4V7_BOOST 5V0 UART_TX 60VIN 3V3_ALWAYS_ON UART_RX EBL 4V0_MODEM 3V3_ANT 60V CAN_250_H CAN_250_L CAN_500_H CAN_500_L IM_OUT GPIO_5 GPIO_1 TAMPER_CONN SWDIO SWDCLK VCU_SWDIO VCU_SWCLK GPIO_2 GPIO_3 GPIO_4 AIN_100V GND BTAT FOR ROAM EXT-BTN VBAT FOR BLACK"
- note added: "Test_PIN TP1 TP2 TP3 TP4 TP5 TP6 TP7 TP8 TP10 J7-1 J7-2 J7-3 J7-4 J7-5 J7-6 J7-7 J7-8 J7-9 J7-10 J7-11 J7-12 J7-13 J7-14 J7-15 J7-16 J7-17 J7-18 TBAT J10-2 J10-1"
- note removed: "Pin_Description 4V7_BOOST 5V0 UART_TX 60VIN 3V3_ALWAYS_ON UART_RX EBL 4V0_MODEM 3V3_ANT 60V CAN_250_H CAN_250_L CAN_500_H CAN_500_L IM_OUT GPIO_5 GPIO_1 TAMPER_CONN SWDIO SWDCLK VCU_SWDIO VCU_SWCLK GPIO_2 GPIO_3 GPIO_4 AIN_100V GND"
- note removed: "Test_PIN TP1 TP2 TP3 TP4 TP5 TP6 TP7 TP8 TP10 J7-1 J7-2 J7-3 J7-4 J7-5 J7-6 J7-7 J7-8 J7-9 J7-10 J7-11 J7-12 J7-13 J7-14 J7-15 J7-16 J7-17 J7-18"
- moved on the sheet: J18, J19
